Commit message: Prune repository to OpenManipulator-X project baseline
- Keep only the classic OpenManipulator-X packages.
- Remove OMX/OMY variants, Gazebo, RealSense, GUI, playground,
  self-collision, and leader/follower controllers.
- Simplify bringup, demos, teleop, and package metadata.
- Remove the old course Docker/CI/docs.
- Add a project README and NOTICE.

File: open_manipulator_description/ros2_control/open_manipulator_x_position.ros2_control.xacro (robot description, xacro)
@@ -3,18 +3,12 @@
   <xacro:macro name="open_manipulator_x_system" params="name prefix port_name:=^|/dev/ttyUSB0 use_sim:=^|false use_fake_hardware:=^|false fake_sensor_commands:=^|false">
     <ros2_control name="${name}" type="system">
-      <xacro:if value="$(arg use_sim)">
-        <hardware>
-          <plugin>gz_ros2_control/GazeboSimSystem</plugin>
-        </hardware>
-      </xacro:if>
-      <xacro:unless value="$(arg use_sim)">
-        <hardware>
-          <xacro:if value="${use_fake_hardware}">
-            <plugin>mock_components/GenericSystem</plugin>
-            <param name="fake_sensor_commands">${fake_sensor_commands}</param>
-            <param name="state_following_offset">0.0</param>
-          </xacro:if>
-          <xacro:unless value="${use_fake_hardware}">
-            <plugin>dynamixel_hardware_interface/DynamixelHardware</plugin>
+      <hardware>
+        <xacro:if value="${use_fake_hardware}">
+          <plugin>mock_components/GenericSystem</plugin>
+          <param name="fake_sensor_commands">${fake_sensor_commands}</param>
+          <param name="state_following_offset">0.0</param>
+        </xacro:if>
+        <xacro:unless value="${use_fake_hardware}">
+          <plugin>dynamixel_hardware_interface/DynamixelHardware</plugin>
             <param name="port_name">${port_name}</param>
             <param name="baud_rate">1000000</param>
@@ -50,7 +44,6 @@
             <param name="prismatic_max">0.019</param>
             <param name="prismatic_min">-0.01</param>
-          </xacro:unless>
-        </hardware>
-      </xacro:unless>
+        </xacro:unless>
+      </hardware>
       <joint name="${prefix}joint1">
         <command_interface name="position"/>
@@ -83,13 +76,4 @@
         <state_interface name="effort"/>
       </joint>
-      <xacro:if value="$(arg use_sim)">
-        <joint name="${prefix}gripper_right_joint">
-          <param name="mimic">${prefix}gripper_left_joint</param>
-          <param name="multiplier">1</param>
-          <state_interface name="position"/>
-          <state_interface name="velocity"/>
-          <state_interface name="effort"/>
-        </joint>
-      </xacro:if>
       <gpio name="dxl1">
         <param name="type">dxl</param>

File: open_manipulator_description/urdf/open_manipulator_x/open_manipulator_x.urdf.xacro (robot description, xacro)
@@ -7,5 +7,4 @@
   <xacro:arg name="port_name" default="/dev/ttyUSB0" />
   <xacro:arg name="ros2_control_type" default="open_manipulator_x_position" />
-  <xacro:include filename="$(find open_manipulator_description)/gazebo/open_manipulator_x.gazebo.xacro" />
   <xacro:include filename="$(find open_manipulator_description)/urdf/open_manipulator_x/open_manipulator_x_arm.urdf.xacro" />
   <xacro:include filename="$(find open_manipulator_description)/ros2_control/$(arg ros2_control_type).ros2_control.xacro" />
@@ -33,9 +32,9 @@
     <origin xyz="0 0 0" rpy="1.5708 0 0"/>
   </joint>
-  <!-- Link OMX on top of the platform -->
+  <!-- Mount the OpenManipulator-X on top of the platform -->
   <joint name="base_to_arm" type="fixed">
     <parent link="base_link"/>
     <child link="$(arg prefix)link1"/>
-    <!-- Position OMX in the right spot on top of the platform -->
+    <!-- Position the OpenManipulator-X on top of the platform -->
     <origin xyz="0 0.025 -0.1263" rpy="-1.5708 -1.5708 0"/>
   </joint>
@@ -57,5 +56,4 @@
   </link>
   <xacro:open_manipulator_x prefix="$(arg prefix)" />
-  <xacro:open_manipulator_x_gazebo prefix="$(arg prefix)" />
   <xacro:open_manipulator_x_system
     name="OpenManipulatorXSystem" prefix="$(arg prefix)" use_sim="$(arg use_sim)"
@@ -63,8 +61,3 @@
     fake_sensor_commands="$(arg fake_sensor_commands)"
     port_name="$(arg port_name)"/>
-  <gazebo>
-    <plugin filename="gz_ros2_control-system" name="gz_ros2_control::GazeboSimROS2ControlPlugin">
-      <parameters>$(find open_manipulator_bringup)/config/open_manipulator_x/hardware_controller_manager.yaml</parameters>
-    </plugin>
-  </gazebo>
 </robot>
